File: discipline-pcb.kicad_pcb (KiCad board)
At the start: 2 copper layers, 304.9 x 122.8 mm, 180 parts, among them J1 AVR-ISP-6, SW1 KEYSW, SW10 KEYSW, SW11 KEYSW, SW12 KEYSW, SW13 KEYSW, SW14 KEYSW, SW15 KEYSW, SW16 KEYSW, SW17 KEYSW, SW18 KEYSW, SW19 KEYSW, SW2 KEYSW, SW20 KEYSW, SW21 KEYSW, SW22 KEYSW, SW23 KEYSW, SW24 KEYSW, SW25 KEYSW, SW26 KEYSW, SW27 KEYSW, SW28 KEYSW, SW29 KEYSW, SW3 KEYSW, SW30 KEYSW, SW31 KEYSW, SW32 KEYSW, SW33 KEYSW, SW34 KEYSW, SW35 KEYSW, SW36 KEYSW, SW37 KEYSW, SW38 KEYSW, SW39 KEYSW, SW4 KEYSW, SW40 KEYSW, SW41 KEYSW, SW42 KEYSW, SW43 KEYSW, SW44 KEYSW, SW45 KEYSW, SW46 KEYSW, SW47 KEYSW, SW48 KEYSW, SW49 KEYSW, SW5 KEYSW, SW50 KEYSW, SW51 KEYSW, SW52 KEYSW, SW53 KEYSW, SW54 KEYSW, SW55 KEYSW, SW56 KEYSW, SW57 KEYSW, SW58 KEYSW, SW59 KEYSW, SW6 KEYSW, SW60 KEYSW, SW61 KEYSW, SW62 KEYSW, SW63 KEYSW, SW64 KEYSW, SW65 KEYSW, SW66 KEYSW, SW67 KEYSW, SW68 KEYSW, SW69 KEYSW, SW7 KEYSW, SW70 KEYSW, SW71 KEYSW, SW72 KEYSW, SW73 KEYSW, SW74 KEYSW, SW8 KEYSW, SW9 KEYSW, U1 ATmega32A-PU, Y1 Crystal

Commit message: Replace USB-C header with TYPE-C-31-M-12
Parts:
- USB1: value USB_C_GCT_USB4085 -> HRO-TYPE-C-31-M-12; footprint cftkb:USB_C_GCT_USB4085 -> Type-C:HRO-TYPE-C-31-M-12-HandSoldering
- moved USB1 2.63 mm to (277.5, 57.7)
Routing:
- net GND: track 241.1 -> 144.4 mm, vias 36 -> 34
- net Net-(D70-Pad1): track 35.9 -> 24.1 mm
- net Net-(D69-Pad1): track 38.8 -> 28.4 mm, vias 1 -> 0
- net VCC: track 21.9 -> 27.2 mm, vias 2 -> 4
- net Net-(R2-Pad1): track 20.5 -> 17.0 mm
- net boot: track 120.6 -> 123.7 mm
- net Net-(R1-Pad2): track 22.7 -> 25.1 mm
- net +5V: track 147.9 -> 145.7 mm
- net reset: track 128.8 -> 127.8 mm
Other:
- net class 5V added: clearance 0.2, trace_width 0.4, via_dia 0.8, via_drill 0.4
- net class GND added: clearance 0.2, trace_width 0.4, via_dia 0.8, via_drill 0.4
